File: hammar.kicad_sch (KiCad schematic)
At the start: 113 parts, among them J1 Conn_01x08_Female, J10 YMIN, J11 ZMIN, J12 X, J13 Y, J14 Z, J15 E, J2 Conn_02x12_Odd_Even, J3 Z, J5 TEND, J7 TBED, J8 USB_C_Receptacle_USB2.0, J9 XMIN, Q1 Q_NMOS_GDS, Q2 Q_NMOS_GSD, Q3 Q_NMOS_GDS, SW1 SW_MEC_5G, SW2 SW_MEC_5G, U1 A4988, U2 ESP32-S2, U3 A4988, U4 A4988, U5 A4988, U6 3,3v lin, Y1 Crystal_GND24_Small

Commit message: Redesign
Parts:
- removed AE1: Antenna_Shield, MyAntennas:SWRU120B, symbol Device:Antenna_Shield
- removed C11, C14, C5, C8, C9: 100nF, Capacitor_SMD:C_0603_1608Metric, symbol Device:C_Small
- removed C16, C17: 1µF, Capacitor_SMD:C_0603_1608Metric, symbol Device:C_Polarized_Small
- removed C2: 15pF, Capacitor_SMD:C_0603_1608Metric, symbol Device:C_Small
- removed C3: 1pF, Capacitor_SMD:C_0603_1608Metric, symbol Device:C_Small
- removed D5: LED_Small, DIY:LED 0603 reverse mount, symbol Device:LED_Small
- removed J11: ZMIN, Connector_JST:JST_PH_S3B-PH-K_1x03_P2.00mm_Horizontal, symbol Connector:Conn_01x03_Male
- removed J2: Conn_02x12_Odd_Even, Connector_PinHeader_2.54mm:PinHeader_2x12_P2.54mm_Vertical, symbol Connector_Generic:Conn_02x12_Odd_Even
- removed SW2: SW_MEC_5G, Button_Switch_THT:SW_PUSH_6mm, symbol Switch:SW_MEC_5G
- removed U2: ESP32-S2, Package_DFN_QFN:QFN-56-1EP_7x7mm_P0.4mm_EP5.6x5.6mm, symbol Espressif:ESP32-S2
- removed Y1: Crystal_GND24_Small, Crystal:Crystal_SMD_3225-4Pin_3.2x2.5mm, symbol Device:Crystal_GND24_Small
- added D5: D_Zener_~3,3v, Diode_SMD:D_SOD-323, symbol Device:D_Zener_Small
- added J11: I2C/SPI, Connector_PinHeader_2.54mm:PinHeader_1x08_P2.54mm_Vertical, symbol Connector:Conn_01x08_Male
- added J16: UART, Connector_PinHeader_2.54mm:PinHeader_1x04_P2.54mm_Vertical, symbol Connector:Conn_01x04_Male
- added J2: Micro_SD_Card, DIY:microSD, symbol Connector:Micro_SD_Card
- added J4: ZMIN_probe, Connector_PinHeader_2.54mm:PinHeader_1x03_P2.54mm_Vertical, symbol Connector:Conn_01x03_Male
- added J6: Conn_01x03_Male, Connector_PinHeader_2.54mm:PinHeader_1x03_P2.54mm_Vertical, symbol Connector:Conn_01x03_Male
- added Q4, Q5: Q_NPN_BEC, Package_TO_SOT_SMD:SOT-23, symbol Device:Q_NPN_BEC
- added R10: 22Ω, Resistor_SMD:R_0603_1608Metric, symbol Device:R_Small
- added R22, R34: 1kΩ, Resistor_SMD:R_0603_1608Metric, symbol Device:R_Small
- added R39: 680Ω, Resistor_SMD:R_0603_1608Metric, symbol Device:R_Small
- added R40, R41, R42, R43: 10kΩ, Resistor_SMD:R_0603_1608Metric, symbol Device:R_Small
- added U2: ESP32-WROOM-32, RF_Module:ESP32-WROOM-32, symbol RF_Module:ESP32-WROOM-32
- added U7: CH340G, Package_SO:SOIC-16_3.9x9.9mm_P1.27mm, symbol Interface_USB:CH340G
- added Y1: Resonator_Small, DIY:resonator_3,2x1,3, symbol Device:Resonator_Small
- C1: value 15pF -> 100nF
- C15, C29, C30: footprint Capacitor_SMD:C_0603_1608Metric -> Capacitor_SMD:C_0805_2012Metric
- J10, J9: footprint Connector_JST:JST_PH_S3B-PH-K_1x03_P2.00mm_Horizontal -> Connector_PinHeader_2.54mm:PinHeader_1x03_P2.54mm_Vertical
- J12, J13, J14, J15: footprint Connector_JST:JST_PH_S4B-PH-K_1x04_P2.00mm_Horizontal -> Connector_PinHeader_2.54mm:PinHeader_1x04_P2.54mm_Vertical
- J3: footprint Connector_JST:JST_PH_B4B-PH-K_1x04_P2.00mm_Vertical -> Connector_PinHeader_2.54mm:PinHeader_1x04_P2.54mm_Vertical
- J5, J7: footprint Connector_JST:JST_PH_S2B-PH-K_1x02_P2.00mm_Horizontal -> Connector_PinHeader_2.54mm:PinHeader_1x02_P2.54mm_Vertical
- R11: value 10kΩ -> 1kΩ
- R26: value 1kΩ -> 10kΩ
- R4: value 10kΩ -> 22Ω
- U6: footprint Package_TO_SOT_SMD:TO-252-2 -> DIY:mini BUCK
Connections:
- net +3.3V: now also C1.2, J11.1 (Pin_1), J16.1 (Pin_1), J2.4 (VDD), J6.1 (Pin_1), R42.2, R43.1, U2.2 (VDD), U7.16 (VCC), U7.4 (V3); no longer R11.2, R4.1
- net +VDC: now also J6.3 (Pin_3); no longer J1.3 (Pin_3)
- net BED: now also U2.26 (IO4)
- net BEDCONN: now also J1.3 (Pin_3); no longer J1.4 (Pin_4)
- net BEDCONN-F: now also J1.4 (Pin_4); no longer F2.2
- net D+: now also R4.2
- net D-: now also R10.1
- net E-DIR: now also U2.28 (IO17)
- net E-EN: now also U2.10 (IO25); no longer R4.2
- net E-STP: now also U2.27 (IO16)
- net END: now also U2.24 (IO2)
- net FAN: now also U2.16 (IO13)
- net GND: now also D5.2 (A), J11.2 (Pin_2), J16.2 (Pin_2), J2.6 (VSS), J4.2 (Pin_2), U2.1 (GND), U2.15 (GND), U2.38 (GND), U2.39 (GND), U7.1 (GND), Y1.2
- net RST: now also Q4.3 (C), R34.1, U2.3 (EN); no longer C22.2, R15.2, SW1.1 (A), SW1.2 (A)
- net T-BED: now also U2.5 (SENSOR_VN)
- net T-END: now also U2.4 (SENSOR_VP)
- net VIN: now also F2.2
- net X-DIR: now also U2.11 (IO26)
- net X-MIN: now also U2.6 (IO34)
- net X-STP: now also U2.12 (IO27)
- net Y-DIR: now also U2.8 (IO32)
- net Y-MIN: now also U2.7 (IO35)
- net Y-STP: now also U2.9 (IO33)
- net Z-DIR: now also R26.2, U2.14 (IO12)
- net Z-MIN: now also D5.1 (K), R39.2, U2.23 (IO15)
- net Z-STP: now also U2.13 (IO14)
- net TX: now reaches R11.1
- net TX: now also J16.4 (Pin_4), U2.34 (RXD0/IO3)
- new net: R10.2, U7.6 (UD-)
- new net: R11.2, U7.2 (TXD)
- new net: R22.1, U7.3 (RXD)
- new net: R4.1, U7.5 (UD+)
- new net: U7.7 (XI), Y1.1
- new net: U7.8 (XO), Y1.3
- new net: C22.2, R15.2, R34.2, SW1.1 (A), SW1.2 (A)
- new net: J4.1 (Pin_1), J6.2 (Pin_2)
- new net: J4.3 (Pin_3), R39.1
- new net: Q4.1 (B), R40.1
- new net: Q5.1 (B), R41.2
- new net DTR: Q5.2 (E), R40.2, U7.13 (~{DTR})
- new net IO0: J11.8 (Pin_8), Q5.3 (C), U2.25 (IO0)
- new net MISO: J11.6 (Pin_6), J2.7 (DAT0), U2.31 (IO19)
- new net MOSI: J11.5 (Pin_5), J2.3 (CMD), U2.37 (IO23)
- new net RTS: Q4.2 (E), R41.1, U7.14 (~{RTS})
- new net RX: J16.3 (Pin_3), R22.2, U2.35 (TXD0/IO1)
- new net SCK: J11.7 (Pin_7), J2.5 (CLK), U2.30 (IO18)
- new net SCL: J11.3 (Pin_3), R42.1, U2.36 (IO22)
- new net SDA: J11.4 (Pin_4), R43.2, U2.33 (IO21)
- new net SS: J2.2 (DAT3/CD), U2.29 (IO5)
- no-connect marks 16 -> 17
Other:
- note added: "USB port"
- note added: "USB reset"
- note added: "aux communication"
- note added: "limit switches"
- note added: "motor connectors"
- note added: "reset switch"
- note added: "screw terminal"
- note added: "stepper drivers"
- note added: "thermistors"
- moved on the sheet: C12, C15, C22, C29, C30, D4, J10, J12, J13, J14, J15, J3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

Commit message: changed designators and updated BOM
Parts:
- D3: renamed from D5; value D_Zener_~3,3v -> Zener_~3,3v
- D6: value D_Small -> USB protection diode, >500mA >24V. Silicon fine
- F1, F2: value Fuse_Small -> 15A Mini fuse + Keystone 3557 fuse holders, or equivalent
- F3: value Polyfuse_Small -> Polyfuse 500mA
- J1: value Conn_01x08_Female -> 8x screw terminal, 5,08mm spacing. rated for >20A
- J10: renamed from J7; value TBED -> 1x2
- J11: renamed from J16; value UART -> 1x4
- J12: renamed from J6; value Conn_01x03_Male -> 1x3
- J13: renamed from J11; value I2C/SPI -> 1x8
- J14: renamed from J9; value XMIN -> 1x3
- J15: renamed from J4; value ZMIN_probe -> 1x3
- J16: renamed from J10; value YMIN -> 1x3
- J2: value Micro_SD_Card -> Micro_SD_Holder
- J4: renamed from J12; value X -> 1x4
- J5: renamed from J13; value Y -> 1x4
- J6: renamed from J14; value Z -> 1x4
- J7: renamed from J15; value E -> 1x4
- J8: renamed from J3; value Z -> 1x4
- J9: renamed from J5; value TEND -> 1x2
- Q1: renamed from Q5; value Q_NPN_BEC -> S9014 or equivalent
- Q2: renamed from Q4; value Q_NPN_BEC -> S9014 or equivalent
- Q3: renamed from Q2; value Q_NMOS_GSD -> TI CSD17310Q5A or equivalent
- Q4: renamed from Q1; value Q_NMOS_GDS -> PMV40UN2R or equivalent
- Q5: renamed from Q3; value Q_NMOS_GDS -> PMV40UN2R or equivalent
- RV1: renamed from RV2; value R_Potentiometer_Small -> Potentiometer_10kΩ
- RV2: renamed from RV4; value R_Potentiometer_Small -> Potentiometer_10kΩ
- RV3: value R_Potentiometer_Small -> Potentiometer_10kΩ
- RV4: renamed from RV1; value R_Potentiometer_Small -> Potentiometer_10kΩ
- RV5, RV6: value Varistor -> ESD varistor, optional
- U5: renamed from U6; value 3,3v lin -> DPAK 3,3v linear regulator + caps OR mini buck converter
- U6: renamed from U2; value ESP32-WROOM-32 -> ESP32-WROOM-32E
- Y1: value Resonator_Small -> Resonator_12mhz
- renumbered C10 to C1, C31 to C10, C26 to C11, C24 to C12, C28 to C13, C36 to C14, C19 to C15, C6 to C16, C33 to C17, C25 to C18, C23 to C19, C35 to C2, C13 to C20, C29 to C21, C30 to C23, C37 to C24, C32 to C25, C15 to C26, C12 to C27, C1 to C28, C21 to C3, C27 to C4, C34 to C5, C20 to C6, C18 to C7, C7 to C8, C4 to C9, D2 to D1, D1 to D2, D3 to D4, D4 to D5, J8 to J3, R37 to R1, R3 to R10, R33 to R11, R21 to R12, R8 to R13, R31 to R14, R18 to R15, R1 to R16, R2 to R17, R17 to R18, R30 to R19, R38 to R2, R7 to R20, R26 to R21, R41 to R22, R40 to R23, R19 to R24, R20 to R25, R29 to R26, R14 to R27, R13 to R28, R34 to R29, R12 to R3, R15 to R30, R32 to R31, R43 to R32, R39 to R33, R42 to R34, R24 to R35, R23 to R36, R25 to R37, R11 to R38, R4 to R39, R16 to R4, R35 to R40, R22 to R41, R10 to R42, R36 to R43, R27 to R7, R28 to R8, U3 to U1, U1 to U2, U5 to U3

Commit message: slight reference update
Other:
- moved on the sheet: D6, F3, J3, R40, R43, RV5, RV6

Commit message: BOM++
Parts:
- R33: value 680Ω -> 10k
Changed lines of the file:
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@@
     (stroke (width 0) (type default) (color 0 0 0 0))
   )
-  (wire (pts (xy 382.27 224.79) (xy 382.27 227.33))
+  (wire (pts (xy 382.27 224.79) (xy 382.27 226.06))
     (stroke (width 0) (type default) (color 0 0 0 0))
   )
@@
     (stroke (width 0) (type default) (color 0 0 0 0))
   )
+  (wire (pts (xy 382.27 231.14) (xy 382.27 233.68))
+    (stroke (width 0) (type default) (color 0 0 0 0))
+  )
   (wire (pts (xy 97.79 274.32) (xy 97.79 275.59))
     (stroke (width 0) (type default) (color 0 0 0 0))
@@
     (stroke (width 0) (type default) (color 0 0 0 0))
   )
-  (wire (pts (xy 382.27 233.68) (xy 382.27 232.41))
-    (stroke (width 0) (type default) (color 0 0 0 0))
-  )
   (wire (pts (xy 353.06 224.79) (xy 353.06 234.95))
     (stroke (width 0) (type default) (color 0 0 0 0))
@@
     (pin "2")
   )
-  (symbol (lib_id "Device:R_Small") (at 382.27 229.87 0) (unit 1)
-    (in_bom yes) (on_board yes)
-    (property "Reference" "R33" (id 0) (at 381 228.6 0)
-      (effects (font (size 1.27 1.27)) (justify right))
-    )
-    (property "Value" "680Ω" (id 1) (at 381 231.14 0)
-      (effects (font (size 1.27 1.27)) (justify right))
-    )
-    (property "Footprint" "Resistor_SMD:R_0603_1608Metric" (id 2) (at 382.27 229.87 0)
-      (effects (font (size 1.27 1.27)) hide)
-    )
-    (property "Datasheet" "~" (id 3) (at 382.27 229.87 0)
-      (effects (font (size 1.27 1.27)) hide)
-    )
-    (pin "1")
-    (pin "2")
-  )
   (symbol (lib_id "Device:R_Small") (at 229.87 27.94 0) (unit 1)
     (in_bom yes) (on_board yes)
@@
     (pin "1")
   )
+  (symbol (lib_id "Device:R_Small") (at 382.27 228.6 0) (unit 1)
+    (in_bom yes) (on_board yes)
+    (property "Reference" "R33" (id 0) (at 381 227.33 0)
+      (effects (font (size 1.27 1.27)) (justify right))
+    )
+    (property "Value" "10k" (id 1) (at 381 229.87 0)
+      (effects (font (size 1.27 1.27)) (justify right))
+    )
+    (property "Footprint" "Resistor_SMD:R_0603_1608Metric" (id 2) (at 382.27 228.6 0)
+      (effects (font (size 1.27 1.27)) hide)
+    )
+    (property "Datasheet" "~" (id 3) (at 382.27 228.6 0)
+      (effects (font (size 1.27 1.27)) hide)
+    )
+    (pin "1")
+    (pin "2")
+  )
   (symbol (lib_id "Device:R_Small") (at 273.05 261.62 180) (unit 1)
     (in_bom yes) (on_board yes)
@@
       (reference "R32") (unit 1) (value "10kΩ") (footprint "Resistor_SMD:R_0603_1608Metric")
     )
-    (path "/31f81989-9b57-4f02-b45c-ef1741cf0df2"
-      (reference "R33") (unit 1) (value "680Ω") (footprint "Resistor_SMD:R_0603_1608Metric")
+    (path "/b56c360d-4c22-478e-8f02-968635d4cfa3"
+      (reference "R33") (unit 1) (value "10k") (footprint "Resistor_SMD:R_0603_1608Metric")
     )
     (path "/536fa290-c4ad-4563-8eae-3e2b761794e3"

Commit message: bom++
Parts:
- R1, R2, R3, R4, R5, R6, R7, R8: value 68mΩ -> 68mΩ shunt
Changed lines of the file:
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@@
       (effects (font (size 1.27 1.27)) (justify left))
     )
-    (property "Value" "68mΩ" (id 1) (at 113.03 71.12 0)
+    (property "Value" "68mΩ shunt" (id 1) (at 113.03 71.12 0)
       (effects (font (size 1.27 1.27)) (justify left))
     )
@@
       (effects (font (size 1.27 1.27)) (justify left))
     )
-    (property "Value" "68mΩ" (id 1) (at 383.54 76.2 0)
+    (property "Value" "68mΩ shunt" (id 1) (at 383.54 76.2 0)
       (effects (font (size 1.27 1.27)) (justify left))
     )
@@
       (effects (font (size 1.27 1.27)) (justify left))
     )
-    (property "Value" "68mΩ" (id 1) (at 303.53 71.12 0)
+    (property "Value" "68mΩ shunt" (id 1) (at 303.53 71.12 0)
       (effects (font (size 1.27 1.27)) (justify left))
     )
@@
       (effects (font (size 1.27 1.27)) (justify left))
     )
-    (property "Value" "68mΩ" (id 1) (at 288.29 76.2 0)
+    (property "Value" "68mΩ shunt" (id 1) (at 288.29 76.2 0)
       (effects (font (size 1.27 1.27)) (justify left))
     )
@@
       (effects (font (size 1.27 1.27)) (justify left))
     )
-    (property "Value" "68mΩ" (id 1) (at 208.28 71.12 0)
+    (property "Value" "68mΩ shunt" (id 1) (at 208.28 71.12 0)
       (effects (font (size 1.27 1.27)) (justify left))
     )
@@
       (effects (font (size 1.27 1.27)) (justify left))
     )
-    (property "Value" "68mΩ" (id 1) (at 398.78 71.12 0)
+    (property "Value" "68mΩ shunt" (id 1) (at 398.78 71.12 0)
       (effects (font (size 1.27 1.27)) (justify left))
     )
@@
       (effects (font (size 1.27 1.27)) (justify left))
     )
-    (property "Value" "68mΩ" (id 1) (at 193.04 76.2 0)
+    (property "Value" "68mΩ shunt" (id 1) (at 193.04 76.2 0)
       (effects (font (size 1.27 1.27)) (justify left))
     )
@@
       (effects (font (size 1.27 1.27)) (justify left))
     )
-    (property "Value" "68mΩ" (id 1) (at 97.79 76.2 0)
+    (property "Value" "68mΩ shunt" (id 1) (at 97.79 76.2 0)
       (effects (font (size 1.27 1.27)) (justify left))
     )
@@
     )
     (path "/40cffe58-622c-446f-a63f-a1c3cedb27c9"
-      (reference "R1") (unit 1) (value "68mΩ") (footprint "Resistor_SMD:R_0603_1608Metric")
+      (reference "R1") (unit 1) (value "68mΩ shunt") (footprint "Resistor_SMD:R_0603_1608Metric")
     )
     (path "/94818848-2d47-4a3a-88ec-7ad52f1c3667"
-      (reference "R2") (unit 1) (value "68mΩ") (footprint "Resistor_SMD:R_0603_1608Metric")
+      (reference "R2") (unit 1) (value "68mΩ shunt") (footprint "Resistor_SMD:R_0603_1608Metric")
     )
     (path "/9ec452b2-9ccb-4e84-9865-41b178afe3ab"
-      (reference "R3") (unit 1) (value "68mΩ") (footprint "Resistor_SMD:R_0603_1608Metric")
+      (reference "R3") (unit 1) (value "68mΩ shunt") (footprint "Resistor_SMD:R_0603_1608Metric")
     )
     (path "/75b74cb3-9860-4f74-9d63-dbc9abf799d8"
-      (reference "R4") (unit 1) (value "68mΩ") (footprint "Resistor_SMD:R_0603_1608Metric")
+      (reference "R4") (unit 1) (value "68mΩ shunt") (footprint "Resistor_SMD:R_0603_1608Metric")
     )
     (path "/dc9cd63d-e670-493d-ab08-2c9a7877bbf0"
-      (reference "R5") (unit 1) (value "68mΩ") (footprint "Resistor_SMD:R_0603_1608Metric")
+      (reference "R5") (unit 1) (value "68mΩ shunt") (footprint "Resistor_SMD:R_0603_1608Metric")
     )
     (path "/10616244-ed1b-4ac4-8c7c-b037e8ca02d0"
-      (reference "R6") (unit 1) (value "68mΩ") (footprint "Resistor_SMD:R_0603_1608Metric")
+      (reference "R6") (unit 1) (value "68mΩ shunt") (footprint "Resistor_SMD:R_0603_1608Metric")
     )
     (path "/709f711e-5d71-4f9e-b309-19bc84206aeb"
-      (reference "R7") (unit 1) (value "68mΩ") (footprint "Resistor_SMD:R_0603_1608Metric")
+      (reference "R7") (unit 1) (value "68mΩ shunt") (footprint "Resistor_SMD:R_0603_1608Metric")
     )
     (path "/65e9748e-24ae-4e8c-b6ba-cd724405d7a6"
-      (reference "R8") (unit 1) (value "68mΩ") (footprint "Resistor_SMD:R_0603_1608Metric")
+      (reference "R8") (unit 1) (value "68mΩ shunt") (footprint "Resistor_SMD:R_0603_1608Metric")
     )
     (path "/83f831cf-6273-4c4e-9aeb-a1807a948f5f"
